File: controller_board/system.sch (EAGLE design)
At the start: 178 parts

Commit message: Pull commit
Parts:
- added R61, R62, R63, R64: (no value), rcl:R-EU_M0805
Connections:
- removed net ENABLE_GATE: U$96G$1.O
- removed net EN_RELAY: JB1.5
- new net N$72: C2.1, R2.2, R61.1, U$68.S
- new net N$73: R61.2, R64.2, U$24G$2.+IN
- new net N$74: C1.1, R1.2, R62.1, U$67.S
- net EN_GATE: now also U$96G$1.O
- net LEM1_M: now also R64.1
- net LEM2_M: now also R63.1
- net N$1: no longer C1.1, R1.2, U$67.S
- net N$4: now also R62.2, R63.2; no longer C2.1, R2.2, U$24G$2.+IN, U$68.S
Other:
- note added: "Driver Enable Circuit"
- note removed: "Enable signal"
- moved on the sheet: C6, C7, U$24G$1, U$24G$2, U$24G$3
